File: hw/fordacp_LCD.kicad_pcb (KiCad board)
At the start: 2 copper layers, 81.9 x 42.4 mm, 35 parts, among them IC1 ATMEGA2560-A, P1 CONN_02X06, U1 SP3485CN, U2 AP1117D50, U3 BLK-MD-SPK-B, U4 XS3860, Y1 16MHz

Commit message: rename XS3868 to S3860M-S
Parts:
- U4: footprint my_modules:XS3868 -> my_modules:S3860M-S
Changed lines of the file:
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@@
-(kicad_pcb (version 4) (host pcbnew 0.201510140731+6267~30~ubuntu14.04.1-product)
+(kicad_pcb (version 4) (host pcbnew 0.201601061458+6427~40~ubuntu14.04.1-stable)
   (general
     (links 108)
     (no_connects 0)
-    (area 182.804999 54.788999 264.870001 97.293501)
+    (area 182.745499 53.69582 264.870001 100.866333)
     (thickness 1.6)
     (drawings 10)
@@
       (net 1 GND))
   )
-  (module my_modules:XS3868 (layer F.Cu)
+  (module my_modules:S3860M-S (layer F.Cu)
     (at 238.9624 84.8616)
     (fp_text reference U4 (at 7.8 -18.7) (layer F.SilkS)
