File: hw/fordacp.sch (KiCad schematic (older format))
At the start: 36 parts, among them IC1 ATMEGA2560-A, P1 CONN_02X06, P2 CONN_02X03, U1 SP3485CN, U2 AP1117D50, U3 BLK-MD-SPK-B, U4 XS3860, Y1 16MHz

Commit message: L1 better housing
Parts:
- added C12, C13: 22, Capacitors_SMD:C_0805, symbol C
Connections:
- wire segments 196 -> 199
Changed lines of the file:
@@
 $EndComp
 $Comp
-L GND #PWR01
+L GND #PWR8
 U 1 1 561E2B62
 P 1850 7350
-F 0 "#PWR01" H 1850 7100 50  0001 C CNN
+F 0 "#PWR8" H 1850 7100 50  0001 C CNN
 F 1 "GND" H 1850 7200 50  0000 C CNN
 F 2 "" H 1850 7350 60  0000 C CNN
@@
 $EndComp
 $Comp
-L +5V #PWR02
+L +5V #PWR9
 U 1 1 561E2EA2
 P 2400 6500
-F 0 "#PWR02" H 2400 6350 50  0001 C CNN
+F 0 "#PWR9" H 2400 6350 50  0001 C CNN
 F 1 "+5V" H 2400 6640 50  0000 C CNN
 F 2 "" H 2400 6500 60  0000 C CNN
@@
 $EndComp
 $Comp
-L +12V #PWR03
+L +12V #PWR2
 U 1 1 561E2EC8
 P 950 6450
-F 0 "#PWR03" H 950 6300 50  0001 C CNN
+F 0 "#PWR2" H 950 6300 50  0001 C CNN
 F 1 "+12V" H 950 6590 50  0000 C CNN
 F 2 "" H 950 6450 60  0000 C CNN
@@
 $EndComp
 $Comp
-L GND #PWR04
+L GND #PWR32
 U 1 1 561E3944
 P 9450 5050
-F 0 "#PWR04" H 9450 4800 50  0001 C CNN
+F 0 "#PWR32" H 9450 4800 50  0001 C CNN
 F 1 "GND" H 9450 4900 50  0000 C CNN
 F 2 "" H 9450 5050 60  0000 C CNN
@@
 ENABLE
 $Comp
-L GNDA #PWR05
+L GNDA #PWR35
 U 1 1 561E3BD2
 P 10200 5050
-F 0 "#PWR05" H 10200 4800 50  0001 C CNN
+F 0 "#PWR35" H 10200 4800 50  0001 C CNN
 F 1 "GNDA" H 10200 4900 50  0000 C CNN
 F 2 "" H 10200 5050 60  0000 C CNN
@@
 AUXINR
 $Comp
-L GNDA #PWR06
+L GNDA #PWR23
 U 1 1 561E4317
 P 8000 1150
-F 0 "#PWR06" H 8000 900 50  0001 C CNN
+F 0 "#PWR23" H 8000 900 50  0001 C CNN
 F 1 "GNDA" H 8000 1000 50  0000 C CNN
 F 2 "" H 8000 1150 60  0000 C CNN
@@
 AUXINR
 $Comp
-L GNDA #PWR07
+L GNDA #PWR27
 U 1 1 561E5090
 P 8400 2750
-F 0 "#PWR07" H 8400 2500 50  0001 C CNN
+F 0 "#PWR27" H 8400 2500 50  0001 C CNN
 F 1 "GNDA" H 8400 2600 50  0000 C CNN
 F 2 "" H 8400 2750 60  0000 C CNN
@@
 AUXINR
 $Comp
-L +12V #PWR08
+L +12V #PWR36
 U 1 1 561E54BC
 P 10750 4450
-F 0 "#PWR08" H 10750 4300 50  0001 C CNN
+F 0 "#PWR36" H 10750 4300 50  0001 C CNN
 F 1 "+12V" H 10750 4590 50  0000 C CNN
 F 2 "" H 10750 4450 60  0000 C CNN
@@
 $EndComp
 $Comp
-L +5V #PWR09
+L +5V #PWR28
 U 1 1 561E6367
 P 8400 3500
-F 0 "#PWR09" H 8400 3350 50  0001 C CNN
+F 0 "#PWR28" H 8400 3350 50  0001 C CNN
 F 1 "+5V" H 8400 3640 50  0000 C CNN
 F 2 "" H 8400 3500 60  0000 C CNN
@@
 $EndComp
 $Comp
-L +5V #PWR010
+L +5V #PWR22
 U 1 1 561E68DF
 P 7950 1850
-F 0 "#PWR010" H 7950 1700 50  0001 C CNN
+F 0 "#PWR22" H 7950 1700 50  0001 C CNN
 F 1 "+5V" H 7950 1990 50  0000 C CNN
 F 2 "" H 7950 1850 60  0000 C CNN
@@
 $EndComp
 $Comp
-L GND #PWR011
+L GND #PWR31
 U 1 1 561E6B56
 P 8900 3800
-F 0 "#PWR011" H 8900 3550 50  0001 C CNN
+F 0 "#PWR31" H 8900 3550 50  0001 C CNN
 F 1 "GND" H 8900 3650 50  0000 C CNN
 F 2 "" H 8900 3800 60  0000 C CNN
@@
 $EndComp
 $Comp
-L GND #PWR012
+L GND #PWR30
 U 1 1 561E6C49
 P 8650 2200
-F 0 "#PWR012" H 8650 1950 50  0001 C CNN
+F 0 "#PWR30" H 8650 1950 50  0001 C CNN
 F 1 "GND" H 8650 2050 50  0000 C CNN
 F 2 "" H 8650 2200 60  0000 C CNN
@@
 MIC
 $Comp
-L GND #PWR013
+L GND #PWR4
 U 1 1 561E8B4F
 P 1600 3800
-F 0 "#PWR013" H 1600 3550 50  0001 C CNN
+F 0 "#PWR4" H 1600 3550 50  0001 C CNN
 F 1 "GND" H 1600 3650 50  0000 C CNN
 F 2 "" H 1600 3800 60  0000 C CNN
@@
 BT_WAKE
 $Comp
-L GND #PWR014
+L GND #PWR3
 U 1 1 561EB2D6
 P 1250 2150
-F 0 "#PWR014" H 1250 1900 50  0001 C CNN
+F 0 "#PWR3" H 1250 1900 50  0001 C CNN
 F 1 "GND" H 1250 2000 50  0000 C CNN
 F 2 "" H 1250 2150 60  0000 C CNN
@@
 $EndComp
 $Comp
-L +5V #PWR015
+L +5V #PWR1
 U 1 1 561EB5E8
 P 950 1800
-F 0 "#PWR015" H 950 1650 50  0001 C CNN
+F 0 "#PWR1" H 950 1650 50  0001 C CNN
 F 1 "+5V" H 950 1940 50  0000 C CNN
 F 2 "" H 950 1800 60  0000 C CNN
@@
 $EndComp
 $Comp
-L GND #PWR016
+L GND #PWR10
 U 1 1 561EB885
 P 2750 2150
-F 0 "#PWR016" H 2750 1900 50  0001 C CNN
+F 0 "#PWR10" H 2750 1900 50  0001 C CNN
 F 1 "GND" H 2750 2000 50  0000 C CNN
 F 2 "" H 2750 2150 60  0000 C CNN
@@
 $EndComp
 $Comp
-L GND #PWR017
+L GND #PWR7
 U 1 1 561EBA36
 P 1850 2700
-F 0 "#PWR017" H 1850 2450 50  0001 C CNN
+F 0 "#PWR7" H 1850 2450 50  0001 C CNN
 F 1 "GND" H 1850 2550 50  0000 C CNN
 F 2 "" H 1850 2700 60  0000 C CNN
@@
 ARD_AREF
 $Comp
-L +5V #PWR018
+L +5V #PWR14
 U 1 1 561F3B87
 P 4700 850
-F 0 "#PWR018" H 4700 700 50  0001 C CNN
+F 0 "#PWR14" H 4700 700 50  0001 C CNN
 F 1 "+5V" H 4700 990 50  0000 C CNN
 F 2 "" H 4700 850 60  0000 C CNN
@@
 $EndComp
 $Comp
-L GND #PWR019
+L GND #PWR6
 U 1 1 561F4EDF
 P 1800 5600
-F 0 "#PWR019" H 1800 5350 50  0001 C CNN
+F 0 "#PWR6" H 1800 5350 50  0001 C CNN
 F 1 "GND" H 1800 5450 50  0000 C CNN
 F 2 "" H 1800 5600 60  0000 C CNN
@@
 $EndComp
 $Comp
-L +5V #PWR020
+L +5V #PWR5
 U 1 1 561F4F9A
 P 1800 4450
-F 0 "#PWR020" H 1800 4300 50  0001 C CNN
+F 0 "#PWR5" H 1800 4300 50  0001 C CNN
 F 1 "+5V" H 1800 4590 50  0000 C CNN
 F 2 "" H 1800 4450 60  0000 C CNN
@@
 $EndComp
 $Comp
-L GND #PWR021
+L GND #PWR29
 U 1 1 561F7E59
 P 8550 6350
-F 0 "#PWR021" H 8550 6100 50  0001 C CNN
+F 0 "#PWR29" H 8550 6100 50  0001 C CNN
 F 1 "GND" H 8550 6200 50  0000 C CNN
 F 2 "" H 8550 6350 60  0000 C CNN
@@
 $EndComp
 $Comp
-L GND #PWR022
+L GND #PWR15
 U 1 1 561F84C6
 P 5200 7100
-F 0 "#PWR022" H 5200 6850 50  0001 C CNN
+F 0 "#PWR15" H 5200 6850 50  0001 C CNN
 F 1 "GND" H 5200 6950 50  0000 C CNN
 F 2 "" H 5200 7100 60  0000 C CNN
@@
 $EndComp
 $Comp
-L GND #PWR023
+L GND #PWR33
 U 1 1 561FBFF0
 P 9750 6250
-F 0 "#PWR023" H 9750 6000 50  0001 C CNN
+F 0 "#PWR33" H 9750 6000 50  0001 C CNN
 F 1 "GND" H 9750 6100 50  0000 C CNN
 F 2 "" H 9750 6250 60  0000 C CNN
@@
 $EndComp
 $Comp
-L GND #PWR024
+L GND #PWR34
 U 1 1 561FC049
 P 10050 6250
-F 0 "#PWR024" H 10050 6000 50  0001 C CNN
+F 0 "#PWR34" H 10050 6000 50  0001 C CNN
 F 1 "GND" H 10050 6100 50  0000 C CNN
 F 2 "" H 10050 6250 60  0000 C CNN
@@
 TX2
 $Comp
-L GND #PWR025
+L GND #PWR37
 U 1 1 562053B0
 P 10800 2200
-F 0 "#PWR025" H 10800 1950 50  0001 C CNN
+F 0 "#PWR37" H 10800 1950 50  0001 C CNN
 F 1 "GND" H 10800 2050 50  0000 C CNN
 F 2 "" H 10800 2200 60  0000 C CNN
@@
 RS485-B
 $Comp
-L GND #PWR026
+L GND #PWR11
 U 1 1 56211668
 P 2850 3850
-F 0 "#PWR026" H 2850 3600 50  0001 C CNN
+F 0 "#PWR11" H 2850 3600 50  0001 C CNN
 F 1 "GND" H 2850 3700 50  0000 C CNN
 F 2 "" H 2850 3850 60  0000 C CNN
@@
 $EndComp
 $Comp
-L +5V #PWR027
+L +5V #PWR19
 U 1 1 5621209A
 P 7450 4000
-F 0 "#PWR027" H 7450 3850 50  0001 C CNN
+F 0 "#PWR19" H 7450 3850 50  0001 C CNN
 F 1 "+5V" H 7450 4140 50  0000 C CNN
 F 2 "" H 7450 4000 60  0000 C CNN
@@
 	3750 1600 3750 1650
 Wire Wire Line
-	3250 1600 3750 1600
+	2950 1600 3750 1600
 Wire Wire Line
 	3250 1600 3250 1650
@@
 Connection ~ 3550 1600
 Wire Wire Line
-	3250 1950 3250 2150
+	3250 1950 3250 2200
 Wire Wire Line
 	3750 1950 3750 2150
@@
 	8250 5350 8250 5500
 $Comp
-L GND #PWR028
+L GND #PWR26
 U 1 1 56223162
 P 8250 5500
-F 0 "#PWR028" H 8250 5250 50  0001 C CNN
+F 0 "#PWR26" H 8250 5250 50  0001 C CNN
 F 1 "GND" H 8250 5350 50  0000 C CNN
 F 2 "" H 8250 5500 60  0000 C CNN
@@
 $EndComp
 $Comp
-L +5V #PWR029
+L +5V #PWR25
 U 1 1 562285BA
 P 8250 4850
-F 0 "#PWR029" H 8250 4700 50  0001 C CNN
+F 0 "#PWR25" H 8250 4700 50  0001 C CNN
 F 1 "+5V" H 8250 4990 50  0000 C CNN
 F 2 "" H 8250 4850 60  0000 C CNN
@@
 Connection ~ 7500 2700
 $Comp
-L GND #PWR030
+L GND #PWR20
 U 1 1 5622ADF9
 P 7500 3200
-F 0 "#PWR030" H 7500 2950 50  0001 C CNN
+F 0 "#PWR20" H 7500 2950 50  0001 C CNN
 F 1 "GND" H 7500 3050 50  0000 C CNN
 F 2 "" H 7500 3200 60  0000 C CNN
@@
 $EndComp
 $Comp
-L +5V #PWR031
+L +5V #PWR24
 U 1 1 5622AE67
 P 8000 2650
-F 0 "#PWR031" H 8000 2500 50  0001 C CNN
+F 0 "#PWR24" H 8000 2500 50  0001 C CNN
 F 1 "+5V" H 8000 2790 50  0000 C CNN
 F 2 "" H 8000 2650 60  0000 C CNN
@@
 Connection ~ 7200 1650
 $Comp
-L GND #PWR032
+L GND #PWR16
 U 1 1 5622B3A5
 P 7200 2150
-F 0 "#PWR032" H 7200 1900 50  0001 C CNN
+F 0 "#PWR16" H 7200 1900 50  0001 C CNN
 F 1 "GND" H 7200 2000 50  0000 C CNN
 F 2 "" H 7200 2150 60  0000 C CNN
@@
 $EndComp
 $Comp
-L +5V #PWR033
+L +5V #PWR21
 U 1 1 5622B3AB
 P 7700 1600
-F 0 "#PWR033" H 7700 1450 50  0001 C CNN
+F 0 "#PWR21" H 7700 1450 50  0001 C CNN
 F 1 "+5V" H 7700 1740 50  0000 C CNN
 F 2 "" H 7700 1600 60  0000 C CNN
@@
 ARD_RESET
 $Comp
-L +5V #PWR034
+L +5V #PWR17
 U 1 1 564F125C
 P 7450 700
-F 0 "#PWR034" H 7450 550 50  0001 C CNN
+F 0 "#PWR17" H 7450 550 50  0001 C CNN
 F 1 "+5V" H 7450 840 50  0000 C CNN
 F 2 "" H 7450 700 60  0000 C CNN
@@
 	7450 800  7450 700
 $Comp
-L GND #PWR035
+L GND #PWR18
 U 1 1 564F1C90
 P 7450 1100
-F 0 "#PWR035" H 7450 850 50  0001 C CNN
+F 0 "#PWR18" H 7450 850 50  0001 C CNN
 F 1 "GND" H 7450 950 50  0000 C CNN
 F 2 "" H 7450 1100 60  0000 C CNN
@@
 Text Label 7450 900  2    60   ~ 0
 MOSI
+$Comp
+L C C12
+U 1 1 565743CA
+P 2950 2350
+F 0 "C12" H 2975 2450 50  0000 L CNN
+F 1 "22" H 2975 2250 50  0000 L CNN
+F 2 "Capacitors_SMD:C_0805" H 2988 2200 30  0001 C CNN
+F 3 "" H 2950 2350 60  0000 C CNN
+	1    2950 2350
+	1    0    0    -1
+$EndComp
+$Comp
+L C C13
+U 1 1 565744F8
+P 3250 2350
+F 0 "C13" H 3275 2450 50  0000 L CNN
+F 1 "22" H 3275 2250 50  0000 L CNN
+F 2 "Capacitors_SMD:C_0805" H 3288 2200 30  0001 C CNN
+F 3 "" H 3250 2350 60  0000 C CNN
+	1    3250 2350
+	1    0    0    -1
+$EndComp
+$Comp
+L GND #PWR12
+U 1 1 56574598
+P 2950 2600
+F 0 "#PWR12" H 2950 2350 50  0001 C CNN
+F 1 "GND" H 2950 2450 50  0000 C CNN
+F 2 "" H 2950 2600 60  0000 C CNN
+F 3 "" H 2950 2600 60  0000 C CNN
+	1    2950 2600
+	1    0    0    -1
+$EndComp
+$Comp
+L GND #PWR13
+U 1 1 56574615
+P 3250 2600
+F 0 "#PWR13" H 3250 2350 50  0001 C CNN
+F 1 "GND" H 3250 2450 50  0000 C CNN
+F 2 "" H 3250 2600 60  0000 C CNN
+F 3 "" H 3250 2600 60  0000 C CNN
+	1    3250 2600
+	1    0    0    -1
+$EndComp
+Wire Wire Line
+	3250 2600 3250 2500
+Wire Wire Line
+	2950 2600 2950 2500
+Wire Wire Line
+	2950 2200 2950 1600
+Connection ~ 3250 1600
+Connection ~ 3250 2150
 $EndSCHEMATC

Commit message: rename xs3860 to xs3868
Parts:
- U4: value XS3860 -> XS3868; symbol XS3860 -> XS3868
Changed lines of the file:
@@
 LIBS:valves
 LIBS:BLK-MD-SPK-B
-LIBS:XS3860
+LIBS:XS3868
 LIBS:fordacp-cache
 EELAYER 25 0
@@
 $EndComp
 $Comp
-L XS3860 U4
+L XS3868 U4
 U 1 1 561E2723
 P 9800 3100
 F 0 "U4" H 9800 3600 60  0000 C CNN
-F 1 "XS3860" H 9800 3700 60  0000 C CNN
+F 1 "XS3868" H 9800 3700 60  0000 C CNN
 F 2 "my_modules:XS3868" H 9800 2300 60  0001 C CNN
 F 3 "" H 9850 3100 60  0000 C CNN

Commit message: rename XS3868 to S3860M-S
Parts:
- U4: value XS3868 -> S3860M-S; footprint my_modules:XS3868 -> my_modules:S3860M-S; symbol XS3868 -> S3860M-S
Changed lines of the file:
@@
 LIBS:valves
 LIBS:BLK-MD-SPK-B
-LIBS:XS3868
+LIBS:S3860M-S
 LIBS:fordacp-cache
 EELAYER 25 0
@@
 $EndComp
 $Comp
-L XS3868 U4
+L S3860M-S U4
 U 1 1 561E2723
 P 9800 3100
 F 0 "U4" H 9800 3600 60  0000 C CNN
-F 1 "XS3868" H 9800 3700 60  0000 C CNN
-F 2 "my_modules:XS3868" H 9800 2300 60  0001 C CNN
+F 1 "S3860M-S" H 9800 3700 60  0000 C CNN
+F 2 "my_modules:S3860M-S" H 9800 2300 60  0001 C CNN
 F 3 "" H 9850 3100 60  0000 C CNN
 	1    9800 3100

Commit message: differential output amplifier with LM358
Parts:
- added C? (x4): 10m/25V, Capacitors_SMD:c_elec_5x5.8, symbol CP
- added C? (x4): 33p, Capacitors_SMD:C_0805_HandSoldering, symbol C
- added C? (x2): 47m/16V, Capacitors_SMD:c_elec_6.3x5.7, symbol CP
- added C? (x2): 100n, Capacitors_SMD:C_0805_HandSoldering, symbol C
- added C?: 2u2, Capacitors_Tantalum_SMD:TantalC_SizeA_EIA-3216_HandSoldering, symbol CP
- added R? (x4): 22k, Resistors_SMD:R_0805_HandSoldering, symbol R
- added R? (x2): 43k, Resistors_SMD:R_0805_HandSoldering, symbol R
- added R? (x2): 30k, Resistors_SMD:R_0805_HandSoldering, symbol R
- added R? (x2): 47k, Resistors_SMD:R_0805_HandSoldering, symbol R
- added R? (x2): 39, Resistors_SMD:R_0805_HandSoldering, symbol R
- added R? (x2): 100k, Resistors_SMD:R_0805_HandSoldering, symbol R
- added U? (x2): LM358, symbol LM358
Connections:
- net +5V: now also R?.2, U?.8 (V+), U?.8 (V+)
- net AUXINL: no longer P1.9 (P9), U4.3 (AOL)
- net AUXINR: no longer P1.11 (P11), U4.4 (AOR)
- net GND: now also P1.10 (P10), P1.12 (P12), C?.1, C?.1, C?.2, R?.1, R?.1, R?.1, U?.4 (V-), U?.4 (V-)
- net GNDA: no longer P1.10 (P10), P1.12 (P12), U4.2 (AOM)
- new net: C?.1, C?.2, R?.2, U?.1
- new net: C?.1, R?.1, R?.2, U?.2 (-)
- new net: C?.2, R?.2, R?.2, U?.3 (+)
- new net: C?.1, R?.1 (x2)
- new net: C?.2, R?.1 (x4)
- new net: C?.2, R?.2, R?.2, U?.5 (+)
- new net: C?.1, R?.1, R?.2, U?.6 (-)
- new net: C?.1, C?.2, R?.2, U?.7
- new net AOUTL: C?.2, C?.2, R?.2, R?.2, R?.2, R?.2
- new net BTAOUTGND: C?.2, C?.2, U4.2 (AOM)
- new net BTAOUTL: C?.1, C?.1, U4.3 (AOL)
- new net BTAOUTR: U4.4 (AOR)
- new net VAGND: C?.1, C?.1, C?.1, R?.1, R?.1, R?.1, R?.2

Commit message: latest modification, I do not remember what it is ...
Parts:
- RV1: symbol POT -> POT-RESCUE-fordacp
Connections:
- net BT_RX: no longer U3.20 (RXD)
Changed lines of the file:
@@
 EESchema Schematic File Version 2
+LIBS:fordacp-rescue
 LIBS:power
 LIBS:device
@@
 	1    0    0    -1
 $EndComp
-Text Label 11150 1450 2    60   ~ 0
+Text Label 11200 1450 2    60   ~ 0
 BT_RX
-Text Label 11150 1550 2    60   ~ 0
+Text Label 11200 1550 2    60   ~ 0
 BT_TX
 Text Label 10800 3050 2    60   ~ 0
@@
 Text Label 10800 3150 2    60   ~ 0
 BT_TX
-Text Label 11150 1650 2    60   ~ 0
+Text Label 11200 1650 2    60   ~ 0
 BT_RST
 Text Label 10800 3450 2    60   ~ 0
@@
 Text Label 8250 1850 0    60   ~ 0
 LED2
-Text Label 11150 1950 2    60   ~ 0
+Text Label 11200 1950 2    60   ~ 0
 BT_WAKE
 $Comp
@@
 $EndComp
 $Comp
-L POT RV1
+L POT-RESCUE-fordacp RV1
 U 1 1 561EB8B0
 P 1450 2650
@@
 	10750 1450 11150 1450
 Wire Wire Line
-	11150 1550 10750 1550
+	10750 1550 11200 1550
 Wire Wire Line
 	10400 3050 10800 3050
@@
 	10800 3150 10400 3150
 Wire Wire Line
-	10750 1650 11150 1650
+	10750 1650 11200 1650
 Wire Wire Line
 	10400 3450 10800 3450
@@
 	8250 1850 8800 1850
 Wire Wire Line
-	10750 1950 11150 1950
+	10750 1950 11200 1950
 Wire Wire Line
 	1250 2150 1250 1850
